File: kicad/Esp32-Weather-EPD/Esp32-Weather-EPD.kicad_pcb (KiCad board)
At the start: 2 copper layers, 130 x 80.3 mm, 16 parts, among them J2 PINHD_1x4_Female, J3 PINHD_1x8_Male

Commit message: refactoring
Parts:
- removed U1: ~, Sephiroth:Waveshare E-Paper Driver Board Rev.3 - ESP32
- added ESP32-EPAPER-BOARD-REV3_1: ~, Sephiroth:Waveshare E-Paper Driver Board Rev.3 - ESP32, F.Cu at (58.9, 112.6)
- moved J3 142.2 mm to (38.4, -23.6), turned to 0 degrees
Routing:
- net /SDA: track 158.3 -> 0.00 mm, vias 2 -> 0
- net /SCL: track 147.8 -> 0.00 mm, vias 4 -> 0
- net /3v3: track 135.2 -> 0.00 mm
- net GND1: track 123.4 -> 0.00 mm
- net /RST: track 115.5 -> 0.00 mm, vias 2 -> 0
- net /BSY: track 111.1 -> 0.00 mm
- net /DC: track 107.0 -> 0.00 mm, vias 2 -> 0
- net /SCK: track 105.2 -> 0.00 mm
- net /CS: track 96.9 -> 0.00 mm
- net Net-(C1-Pad1): track 91.2 -> 0.00 mm, vias 2 -> 0
- net /SDI: track 89.5 -> 0.00 mm
- net +4V: track 30.0 -> 0.00 mm
- net Net-(ESP32-EPAPER-BOARD-REV3_1-~{EN}): track 10.3 -> 0.00 mm
